Commit message: Update upper_rails.urdf.xacro

File: ur_components_description/urdf/upper_rails.urdf.xacro (robot description, xacro)
@@ -1,6 +1,5 @@
 <?xml version="1.0"?>
 <robot xmlns:xacro="http://www.ros.org/wiki/xacro">
-  <xacro:macro name="upper_rails"
-    params="parent_link xyz rpy">
+  <xacro:macro name="upper_rails" params="parent_link xyz rpy">
     <link name="upper_rails_link">
       <collision>
