Commit message: Update ur_components_description/urdf/zed2i.urdf.xacro
Co-authored-by: Dawid Kmak <73443304+KmakD@users.noreply.github.com>

File: ur_components_description/urdf/zed2i.urdf.xacro (robot description, xacro)
@@ -53,5 +53,5 @@
       <parent link="zed2i_camera_center" />
       <child link="zed2i_mag_link" />
-      <origin xyz="0 0 0" rpy="0 0 0" />
+      <origin xyz="0.0 0.0 0.0" rpy="0.0 0.0 0.0" />
     </joint>
     <link name="zed2i_baro_link" />

Commit message: Update ur_components_description/urdf/zed2i.urdf.xacro
Co-authored-by: Dawid Kmak <73443304+KmakD@users.noreply.github.com>

File: ur_components_description/urdf/zed2i.urdf.xacro (robot description, xacro)
@@ -59,5 +59,5 @@
       <parent link="zed2i_camera_center" />
       <child link="zed2i_baro_link" />
-      <origin xyz="0 0 0" rpy="0 0 0" />
+      <origin xyz="0.0 0.0 0.0" rpy="0.0 0.0 0.0" />
     </joint>
     <link name="zed2i_temp_left_link" />

Commit message: Update ur_components_description/urdf/zed2i.urdf.xacro
Co-authored-by: Dawid Kmak <73443304+KmakD@users.noreply.github.com>

File: ur_components_description/urdf/zed2i.urdf.xacro (robot description, xacro)
@@ -65,5 +65,5 @@
       <parent link="zed2i_left_camera_frame" />
       <child link="zed2i_temp_left_link" />
-      <origin xyz="0 0 0" rpy="0 0 0" />
+      <origin xyz="0.0 0.0 0.0" rpy="0.0 0.0 0.0" />
     </joint>
     <link name="zed2i_temp_right_link" />

Commit message: Update ur_components_description/urdf/zed2i.urdf.xacro
Co-authored-by: Dawid Kmak <73443304+KmakD@users.noreply.github.com>

File: ur_components_description/urdf/zed2i.urdf.xacro (robot description, xacro)
@@ -71,5 +71,5 @@
       <parent link="zed2i_right_camera_frame" />
       <child link="zed2i_temp_right_link" />
-      <origin xyz="0 0 0" rpy="0 0 0" />
+      <origin xyz="0.0 0.0 0.0" rpy="0.0 0.0 0.0" />
     </joint>
   </xacro:macro>

Commit message: Update ur_components_description/urdf/zed2i.urdf.xacro
Co-authored-by: Dawid Kmak <73443304+KmakD@users.noreply.github.com>

File: ur_components_description/urdf/zed2i.urdf.xacro (robot description, xacro)
@@ -45,5 +45,5 @@
     <link name="zed2i_right_camera_optical_frame" />
     <joint name="zed2i_right_camera_optical_joint" type="fixed">
-      <origin xyz="-0.01 0 0" rpy="-${pi/2} 0.0 -${pi/2}" />
+      <origin xyz="-0.01 0.0 0.0" rpy="-${pi/2} 0.0 -${pi/2}" />
       <parent link="zed2i_right_camera_frame" />
       <child link="zed2i_right_camera_optical_frame" />
