Commit message: fix meshes

File: ur3_moveit_config/urdf/panther_ur3.urdf.xacro (robot description, xacro)
@@ -7,15 +7,26 @@
   <xacro:include filename="$(find panther_description)/urdf/panther_macro.urdf.xacro" ns="husarion" />
   <xacro:include filename="$(find ur_description)/urdf/inc/ur3_macro.xacro" ns="universal_robot"/>
-  <xacro:husarion.panther_robot dual_bat="$(arg dual_bat)" wheel_config_path="$(arg wheel_config_path)" />
-  <xacro:universal_robot.ur3_robot prefix="panther_ur3_" />
-  <joint name="base_link_to_ur3_link_joint" type="fixed">
-    <origin xyz="-0.095 0.0975 0.375" rpy="0.0 0.0 ${pi/2}" />
-    <parent link="base_link" />
+  <xacro:include filename="$(find ur_components_description)/urdf/mounting_plate.urdf.xacro" ns="mounting_plate" />
+  <xacro:include filename="$(find ur_components_description)/urdf/upper_rails.urdf.xacro" ns="rails" />
+  <xacro:husarion.panther_robot
+    dual_bat="$(arg dual_bat)"
+    wheel_config_path="$(arg wheel_config_path)"
+    use_ros_control="True" />
+  <xacro:rails.upper_rails
+      parent_link="cover_link"
+      xyz="0.0 0.0 -0.02"
+      rpy="0.0 0.0 0.0" />
+  <xacro:mounting_plate.mounting_plate
+    parent_link="upper_rails_link"
+    xyz="-0.095 0.0975 0.05"
+    rpy="0.0 0.0 0.0" />
+  <joint name="ur_mounting_plate_to_ur3_link_joint" type="fixed">
+    <origin xyz="0.0 0.0 0.0" rpy="0.0 0.0 ${pi/2}" />
+    <parent link="ur_mounting_plate_link" />
     <child link="panther_ur3_base_link" />
   </joint>
+  <xacro:universal_robot.ur3_robot prefix="panther_ur3_" />
   <!-- Components -->
   <xacro:include filename="$(find panther_description)/urdf/components/external_antenna.urdf.xacro" ns="antena" />
-  <xacro:include filename="$(find ur_components_description)/urdf/upper_rails.urdf.xacro" ns="rails" />
   <xacro:antena.external_antenna parent_link="base_link" xyz="0.18 0.15 0.377" rpy="0.0 0.0 ${pi}" />
-  <xacro:rails.upper_rails parent_link="base_link" xyz="0.0 0.0 0.334" rpy="0.0 ${-pi/2} 0.0" />
 </robot>

File: ur5e_moveit_config/urdf/panther_ur5e.urdf.xacro (robot description, xacro)
@@ -6,32 +6,49 @@
   <!-- Robot -->
   <xacro:include filename="$(find panther_description)/urdf/panther_macro.urdf.xacro" ns="husarion" />
-  <xacro:include filename="$(find ur_description)/urdf/inc/ur5e_macro.xacro" ns="universal_robot" />
+  <xacro:include filename="$(find ur_description)/urdf/inc/ur5e_macro.xacro" ns="universal_robot"/>
+  <xacro:include filename="$(find ur_components_description)/urdf/mounting_plate.urdf.xacro" ns="mounting_plate" />
+  <xacro:include filename="$(find ur_components_description)/urdf/upper_rails.urdf.xacro" ns="rails" />
   <xacro:husarion.panther_robot
     dual_bat="$(arg dual_bat)"
     wheel_config_path="$(arg wheel_config_path)"
     use_ros_control="True" />
-  <xacro:universal_robot.ur5e_robot prefix="panther_ur5e_" />
-  <joint name="base_link_to_ur5e_link_joint" type="fixed">
-    <origin xyz="-0.095 0.0975 0.375" rpy="0.0 0.0 ${pi/2}" />
-    <parent link="base_link" />
+  <xacro:rails.upper_rails
+      parent_link="cover_link"
+      xyz="0.0 0.0 -0.02"
+      rpy="0.0 0.0 0.0" />
+  <xacro:mounting_plate.mounting_plate
+    parent_link="upper_rails_link"
+    xyz="-0.095 0.0975 0.05"
+    rpy="0.0 0.0 0.0" />
+  <joint name="ur_mounting_plate_to_ur5e_link_joint" type="fixed">
+    <origin xyz="0.0 0.0 0.0" rpy="0.0 0.0 ${pi/2}" />
+    <parent link="ur_mounting_plate_link" />
     <child link="panther_ur5e_base_link" />
   </joint>
+  <xacro:universal_robot.ur5e_robot prefix="panther_ur5e_" />
   <!-- Sensors -->
   <xacro:include filename="$(find ros_components_description)/urdf/velodyne_puck.urdf.xacro"
     ns="velodyne" />
   <xacro:include filename="$(find realsense2_description)/urdf/_d435i.urdf.xacro" ns="rs" />
-  <xacro:velodyne.velodyne_puck parent_link="base_link" xyz="0.05 -0.13 0.527" rpy="0.0 0.0 0.0"
+  <xacro:velodyne.velodyne_puck
+    parent_link="cover_link"
+    xyz="0.05 -0.13 0.15"
+    rpy="0.0 0.0 0.0"
     use_gpu="$(arg use_gpu)" />
-  <xacro:rs.sensor_d435i parent="base_link" use_nominal_extrinsics="true">
-    <origin xyz="0.19 0.05 0.427" rpy="0.0 0.0 0.0" />
+  <xacro:rs.sensor_d435i
+    parent="cover_link"
+    use_nominal_extrinsics="true">
+    <origin xyz="0.19 0.05 0.05" rpy="0.0 0.0 0.0" />
   </xacro:rs.sensor_d435i>
   <!-- Components -->
-  <xacro:include filename="$(find panther_description)/urdf/components/external_antenna.urdf.xacro"
-    ns="antena" />
-  <xacro:include filename="$(find ur_components_description)/urdf/power_supply.urdf.xacro"
-    ns="power_supply" />
-  <xacro:include filename="$(find ur_components_description)/urdf/upper_rails.urdf.xacro" ns="rails" />
-  <xacro:antena.external_antenna parent_link="base_link" xyz="0.18 0.15 0.377" rpy="0.0 0.0 ${pi}" />
-  <xacro:power_supply.power_supply parent_link="base_link" xyz="0.0 -0.13 0.377" rpy="0.0 0.0 0.0" />
-  <xacro:rails.upper_rails parent_link="base_link" xyz="0.0 0.0 0.334" rpy="0.0 ${-pi/2} 0.0" />
+  <xacro:include filename="$(find panther_description)/urdf/components/external_antenna.urdf.xacro" ns="antena" />
+  <xacro:include filename="$(find ur_components_description)/urdf/power_supply.urdf.xacro" ns="power_supply" />
+  <xacro:antena.external_antenna
+    parent_link="cover_link"
+    xyz="0.18 0.15 0.0"
+    rpy="0.0 0.0 ${pi}" />
+  <xacro:power_supply.power_supply
+    parent_link="cover_link"
+    xyz="0.0 -0.13 0.0"
+    rpy="0.0 0.0 0.0" />
 </robot>

File: ur5e_onrobot_rg2_moveit_config/urdf/panther_ur5e_rg2.urdf.xacro (robot description, xacro)
@@ -7,12 +7,30 @@
   <xacro:include filename="$(find panther_description)/urdf/panther_macro.urdf.xacro" ns="husarion" />
   <xacro:include filename="$(find ur_description)/urdf/inc/ur5e_macro.xacro" ns="universal_robot"/>
+  <xacro:include filename="$(find ur_components_description)/urdf/mounting_plate.urdf.xacro" ns="mounting_plate" />
+  <xacro:include filename="$(find onrobot_rg2_description)/urdf/onrobot_rg2.urdf.xacro" ns="gripper" />
   <xacro:include filename="$(find onrobot_rg2_description)/urdf/onrobot_quick_changer.urdf.xacro" ns="changer" />
-  <xacro:include filename="$(find onrobot_rg2_description)/urdf/onrobot_rg2.urdf.xacro" ns="gripper" />
+  <xacro:include filename="$(find ur_components_description)/urdf/upper_rails.urdf.xacro" ns="rails" />
   <xacro:husarion.panther_robot
     dual_bat="$(arg dual_bat)"
     wheel_config_path="$(arg wheel_config_path)"
     use_ros_control="True" />
+  <xacro:rails.upper_rails
+      parent_link="cover_link"
+      xyz="0.0 0.0 -0.02"
+      rpy="0.0 0.0 0.0" />
+  <xacro:mounting_plate.mounting_plate
+    parent_link="upper_rails_link"
+    xyz="0.085 0.0975 0.05"
+    rpy="0.0 0.0 0.0" />
+  <joint name="ur_mounting_plate_to_ur5e_link_joint" type="fixed">
+    <origin xyz="0.0 0.0 0.0" rpy="0.0 0.0 ${pi/2}" />
+    <parent link="ur_mounting_plate_link" />
+    <child link="panther_ur5e_base_link" />
+  </joint>
   <xacro:universal_robot.ur5e_robot prefix="panther_ur5e_" />
-  <xacro:changer.onrobot_quick_changer parent_link="panther_ur5e_tool0" xyz="0.0 0.0 0.0" rpy="0.0 0.0 0.0" />
+  <xacro:changer.onrobot_quick_changer
+    parent_link="panther_ur5e_tool0"
+    xyz="0.0 0.0 0.0"
+    rpy="0.0 0.0 0.0" />
   <xacro:gripper.onrobot_rg2
     parent_link="quick_changer_link"
@@ -20,11 +38,14 @@
     rpy="${-pi/2} ${-pi/2} 0.0"
     use_ros_control="False" />
-  <joint name="base_link_to_ur5e_link_joint" type="fixed">
-    <origin xyz="-0.095 0.0975 0.375" rpy="0.0 0.0 ${pi/2}" />
-    <parent link="base_link" />
-    <child link="panther_ur5e_base_link" />
-  </joint>
   <!-- Components -->
-  <xacro:include filename="$(find ur_components_description)/urdf/upper_rails.urdf.xacro" ns="rails" />
-  <xacro:rails.upper_rails parent_link="base_link" xyz="0.0 0.0 0.334" rpy="0.0 ${-pi/2} 0.0" />
+  <xacro:include filename="$(find ur_components_description)/urdf/zed2i.urdf.xacro" ns="zed" />
+  <xacro:include filename="$(find panther_description)/urdf/components/external_antenna.urdf.xacro" ns="antena" />
+  <xacro:zed.zed2i_camera
+    parent_link="cover_link"
+    xyz="0.19 -0.1 0.05"
+    rpy="0.0 0.0 0.0" />
+  <xacro:antena.external_antenna
+    parent_link="cover_link"
+    xyz="0.18 -0.15 0.0"
+    rpy="0.0 0.0 ${pi}" />
 </robot>

File: ur_components_description/urdf/power_supply.urdf.xacro (robot description, xacro)
@@ -16,9 +16,4 @@
         </geometry>
       </visual>
-      <inertial>
-        <mass value="0.59" />
-        <inertia ixx="0.003964" ixy="0.0" ixz="0.0" iyy="0.0003964" iyz="0.0" izz="0.0004177" />
-        <origin xyz="0.045 0.0 0.0058" rpy="0.0 0.0 0.0" />
-      </inertial>
     </link>
     <joint name="${parent_link}_to_power_supply_link_joint" type="fixed">

File: ur_components_description/urdf/upper_rails.urdf.xacro (robot description, xacro)
@@ -2,23 +2,18 @@
 <robot xmlns:xacro="http://www.ros.org/wiki/xacro">
   <xacro:macro name="upper_rails"
-              params="parent_link xyz rpy">
+    params="parent_link xyz rpy">
     <link name="upper_rails_link">
       <collision>
         <geometry>
-          <mesh filename="file://$(find ur_components_description)/meshes/upper_rails.stl" scale="0.01 0.01 0.01" />
+          <mesh filename="file://$(find ur_components_description)/meshes/upper_rails.stl" />
         </geometry>
-        <origin xyz="0.0 0.0 0.0" rpy=" ${pi/2} 0.0 ${pi/2}" />
+        <origin xyz="0.0 0.0 0.0" rpy=" 0.0 0.0 0.0" />
       </collision>
       <visual>
         <geometry>
-          <mesh filename="file://$(find ur_components_description)/meshes/upper_rails.stl" scale="0.01 0.01 0.01" />
+          <mesh filename="file://$(find ur_components_description)/meshes/upper_rails.dae" />
         </geometry>
-        <origin xyz="0.0 0.0 0.0" rpy=" ${pi/2} 0.0 ${pi/2}" />
-        <material name="Black" />
+        <origin xyz="0.0 0.0 0.0" rpy="0.0 0.0 0.0" />
       </visual>
-      <inertial>
-        <mass value="0.0000001" />
-        <inertia ixx="1.0" ixy="0.0" ixz="0.0" iyy="1.0" iyz="0.0" izz="1.0" />
-      </inertial>
     </link>
     <joint name="${parent_link}_to_upper_rails_link_joint" type="fixed">
@@ -27,7 +22,4 @@
       <child link="upper_rails_link" />
     </joint>
-    <gazebo reference="upper_rails_link">
-      <material>Gazebo/Black</material>
-    </gazebo>
   </xacro:macro>
 </robot>

Commit message: fix meshes (#3)
* fix meshes

* Update ur5e_moveit_config/urdf/panther_ur5e.urdf.xacro

Co-authored-by: Dawid Kmak <73443304+KmakD@users.noreply.github.com>

* Update ur5e_onrobot_rg2_moveit_config/urdf/panther_ur5e_rg2.urdf.xacro

Co-authored-by: Dawid Kmak <73443304+KmakD@users.noreply.github.com>

* Update ur3_moveit_config/urdf/panther_ur3.urdf.xacro

Co-authored-by: Dawid Kmak <73443304+KmakD@users.noreply.github.com>

* Update ur_components_description/urdf/zed2i.urdf.xacro

Co-authored-by: Dawid Kmak <73443304+KmakD@users.noreply.github.com>

* Update ur_components_description/urdf/zed2i.urdf.xacro

Co-authored-by: Dawid Kmak <73443304+KmakD@users.noreply.github.com>

* Update upper_rails.urdf.xacro

* Update ur_components_description/urdf/zed2i.urdf.xacro

Co-authored-by: Dawid Kmak <73443304+KmakD@users.noreply.github.com>

* Update ur_components_description/urdf/zed2i.urdf.xacro

Co-authored-by: Dawid Kmak <73443304+KmakD@users.noreply.github.com>

* Update ur_components_description/urdf/zed2i.urdf.xacro

Co-authored-by: Dawid Kmak <73443304+KmakD@users.noreply.github.com>

* fix poses

---------

Co-authored-by: Dawid Kmak <73443304+KmakD@users.noreply.github.com>

File: ur3_moveit_config/urdf/panther_ur3.urdf.xacro (robot description, xacro)
@@ -6,16 +6,27 @@
   <!-- Robot -->
   <xacro:include filename="$(find panther_description)/urdf/panther_macro.urdf.xacro" ns="husarion" />
-  <xacro:include filename="$(find ur_description)/urdf/inc/ur3_macro.xacro" ns="universal_robot"/>
-  <xacro:husarion.panther_robot dual_bat="$(arg dual_bat)" wheel_config_path="$(arg wheel_config_path)" />
-  <xacro:universal_robot.ur3_robot prefix="panther_ur3_" />
-  <joint name="base_link_to_ur3_link_joint" type="fixed">
-    <origin xyz="-0.095 0.0975 0.375" rpy="0.0 0.0 ${pi/2}" />
-    <parent link="base_link" />
+  <xacro:include filename="$(find ur_description)/urdf/inc/ur3_macro.xacro" ns="universal_robot" />
+  <xacro:include filename="$(find ur_components_description)/urdf/mounting_plate.urdf.xacro" ns="mounting_plate" />
+  <xacro:include filename="$(find ur_components_description)/urdf/upper_rails.urdf.xacro" ns="rails" />
+  <xacro:husarion.panther_robot
+    dual_bat="$(arg dual_bat)"
+    wheel_config_path="$(arg wheel_config_path)"
+    use_ros_control="True" />
+  <xacro:rails.upper_rails
+      parent_link="cover_link"
+      xyz="0.0 0.0 -0.02"
+      rpy="0.0 0.0 0.0" />
+  <xacro:mounting_plate.mounting_plate
+    parent_link="upper_rails_link"
+    xyz="-0.095 0.0975 0.05"
+    rpy="0.0 0.0 0.0" />
+  <joint name="ur_mounting_plate_to_ur3_link_joint" type="fixed">
+    <origin xyz="0.0 0.0 0.0" rpy="0.0 0.0 ${pi/2}" />
+    <parent link="ur_mounting_plate_link" />
     <child link="panther_ur3_base_link" />
   </joint>
+  <xacro:universal_robot.ur3_robot prefix="panther_ur3_" />
   <!-- Components -->
   <xacro:include filename="$(find panther_description)/urdf/components/external_antenna.urdf.xacro" ns="antena" />
-  <xacro:include filename="$(find ur_components_description)/urdf/upper_rails.urdf.xacro" ns="rails" />
-  <xacro:antena.external_antenna parent_link="base_link" xyz="0.18 0.15 0.377" rpy="0.0 0.0 ${pi}" />
-  <xacro:rails.upper_rails parent_link="base_link" xyz="0.0 0.0 0.334" rpy="0.0 ${-pi/2} 0.0" />
+  <xacro:antena.external_antenna parent_link="cover_link" xyz="0.18 0.15 0.02" rpy="0.0 0.0 ${pi}" />
 </robot>

File: ur5e_moveit_config/urdf/panther_ur5e.urdf.xacro (robot description, xacro)
@@ -7,31 +7,48 @@
   <xacro:include filename="$(find panther_description)/urdf/panther_macro.urdf.xacro" ns="husarion" />
   <xacro:include filename="$(find ur_description)/urdf/inc/ur5e_macro.xacro" ns="universal_robot" />
+  <xacro:include filename="$(find ur_components_description)/urdf/mounting_plate.urdf.xacro" ns="mounting_plate" />
+  <xacro:include filename="$(find ur_components_description)/urdf/upper_rails.urdf.xacro" ns="rails" />
   <xacro:husarion.panther_robot
     dual_bat="$(arg dual_bat)"
     wheel_config_path="$(arg wheel_config_path)"
     use_ros_control="True" />
-  <xacro:universal_robot.ur5e_robot prefix="panther_ur5e_" />
-  <joint name="base_link_to_ur5e_link_joint" type="fixed">
-    <origin xyz="-0.095 0.0975 0.375" rpy="0.0 0.0 ${pi/2}" />
-    <parent link="base_link" />
+  <xacro:rails.upper_rails
+      parent_link="cover_link"
+      xyz="0.0 0.0 -0.02"
+      rpy="0.0 0.0 0.0" />
+  <xacro:mounting_plate.mounting_plate
+    parent_link="upper_rails_link"
+    xyz="-0.095 0.0975 0.05"
+    rpy="0.0 0.0 0.0" />
+  <joint name="ur_mounting_plate_to_ur5e_link_joint" type="fixed">
+    <origin xyz="0.0 0.0 0.0" rpy="0.0 0.0 ${pi/2}" />
+    <parent link="ur_mounting_plate_link" />
     <child link="panther_ur5e_base_link" />
   </joint>
+  <xacro:universal_robot.ur5e_robot prefix="panther_ur5e_" />
   <!-- Sensors -->
   <xacro:include filename="$(find ros_components_description)/urdf/velodyne_puck.urdf.xacro"
     ns="velodyne" />
   <xacro:include filename="$(find realsense2_description)/urdf/_d435i.urdf.xacro" ns="rs" />
-  <xacro:velodyne.velodyne_puck parent_link="base_link" xyz="0.05 -0.13 0.527" rpy="0.0 0.0 0.0"
+  <xacro:velodyne.velodyne_puck
+    parent_link="cover_link"
+    xyz="0.05 -0.13 0.17"
+    rpy="0.0 0.0 0.0"
     use_gpu="$(arg use_gpu)" />
-  <xacro:rs.sensor_d435i parent="base_link" use_nominal_extrinsics="true">
-    <origin xyz="0.19 0.05 0.427" rpy="0.0 0.0 0.0" />
+  <xacro:rs.sensor_d435i
+    parent="cover_link"
+    use_nominal_extrinsics="true">
+    <origin xyz="0.19 0.05 0.05" rpy="0.0 0.0 0.0" />
   </xacro:rs.sensor_d435i>
   <!-- Components -->
-  <xacro:include filename="$(find panther_description)/urdf/components/external_antenna.urdf.xacro"
-    ns="antena" />
-  <xacro:include filename="$(find ur_components_description)/urdf/power_supply.urdf.xacro"
-    ns="power_supply" />
-  <xacro:include filename="$(find ur_components_description)/urdf/upper_rails.urdf.xacro" ns="rails" />
-  <xacro:antena.external_antenna parent_link="base_link" xyz="0.18 0.15 0.377" rpy="0.0 0.0 ${pi}" />
-  <xacro:power_supply.power_supply parent_link="base_link" xyz="0.0 -0.13 0.377" rpy="0.0 0.0 0.0" />
-  <xacro:rails.upper_rails parent_link="base_link" xyz="0.0 0.0 0.334" rpy="0.0 ${-pi/2} 0.0" />
+  <xacro:include filename="$(find panther_description)/urdf/components/external_antenna.urdf.xacro" ns="antena" />
+  <xacro:include filename="$(find ur_components_description)/urdf/power_supply.urdf.xacro" ns="power_supply" />
+  <xacro:antena.external_antenna
+    parent_link="cover_link"
+    xyz="0.18 0.15 0.02"
+    rpy="0.0 0.0 ${pi}" />
+  <xacro:power_supply.power_supply
+    parent_link="cover_link"
+    xyz="0.0 -0.13 0.02"
+    rpy="0.0 0.0 0.0" />
 </robot>

File: ur5e_onrobot_rg2_moveit_config/urdf/panther_ur5e_rg2.urdf.xacro (robot description, xacro)
@@ -6,13 +6,31 @@
   <!-- Robot -->
   <xacro:include filename="$(find panther_description)/urdf/panther_macro.urdf.xacro" ns="husarion" />
-  <xacro:include filename="$(find ur_description)/urdf/inc/ur5e_macro.xacro" ns="universal_robot"/>
+  <xacro:include filename="$(find ur_description)/urdf/inc/ur5e_macro.xacro" ns="universal_robot" />
+  <xacro:include filename="$(find ur_components_description)/urdf/mounting_plate.urdf.xacro" ns="mounting_plate" />
+  <xacro:include filename="$(find onrobot_rg2_description)/urdf/onrobot_rg2.urdf.xacro" ns="gripper" />
   <xacro:include filename="$(find onrobot_rg2_description)/urdf/onrobot_quick_changer.urdf.xacro" ns="changer" />
-  <xacro:include filename="$(find onrobot_rg2_description)/urdf/onrobot_rg2.urdf.xacro" ns="gripper" />
+  <xacro:include filename="$(find ur_components_description)/urdf/upper_rails.urdf.xacro" ns="rails" />
   <xacro:husarion.panther_robot
     dual_bat="$(arg dual_bat)"
     wheel_config_path="$(arg wheel_config_path)"
     use_ros_control="True" />
+  <xacro:rails.upper_rails
+      parent_link="cover_link"
+      xyz="0.0 0.0 -0.02"
+      rpy="0.0 0.0 0.0" />
+  <xacro:mounting_plate.mounting_plate
+    parent_link="upper_rails_link"
+    xyz="0.085 0.0975 0.05"
+    rpy="0.0 0.0 0.0" />
+  <joint name="ur_mounting_plate_to_ur5e_link_joint" type="fixed">
+    <origin xyz="0.0 0.0 0.0" rpy="0.0 0.0 ${pi/2}" />
+    <parent link="ur_mounting_plate_link" />
+    <child link="panther_ur5e_base_link" />
+  </joint>
   <xacro:universal_robot.ur5e_robot prefix="panther_ur5e_" />
-  <xacro:changer.onrobot_quick_changer parent_link="panther_ur5e_tool0" xyz="0.0 0.0 0.0" rpy="0.0 0.0 0.0" />
+  <xacro:changer.onrobot_quick_changer
+    parent_link="panther_ur5e_tool0"
+    xyz="0.0 0.0 0.0"
+    rpy="0.0 0.0 0.0" />
   <xacro:gripper.onrobot_rg2
     parent_link="quick_changer_link"
@@ -20,11 +38,14 @@
     rpy="${-pi/2} ${-pi/2} 0.0"
     use_ros_control="False" />
-  <joint name="base_link_to_ur5e_link_joint" type="fixed">
-    <origin xyz="-0.095 0.0975 0.375" rpy="0.0 0.0 ${pi/2}" />
-    <parent link="base_link" />
-    <child link="panther_ur5e_base_link" />
-  </joint>
   <!-- Components -->
-  <xacro:include filename="$(find ur_components_description)/urdf/upper_rails.urdf.xacro" ns="rails" />
-  <xacro:rails.upper_rails parent_link="base_link" xyz="0.0 0.0 0.334" rpy="0.0 ${-pi/2} 0.0" />
+  <xacro:include filename="$(find ur_components_description)/urdf/zed2i.urdf.xacro" ns="zed" />
+  <xacro:include filename="$(find panther_description)/urdf/components/external_antenna.urdf.xacro" ns="antena" />
+  <xacro:zed.zed2i_camera
+    parent_link="cover_link"
+    xyz="0.21 -0.07 0.06"
+    rpy="0.0 0.0 0.0" />
+  <xacro:antena.external_antenna
+    parent_link="cover_link"
+    xyz="0.18 -0.15 0.02"
+    rpy="0.0 0.0 ${pi}" />
 </robot>

File: ur_components_description/urdf/upper_rails.urdf.xacro (robot description, xacro)
@@ -1,24 +1,18 @@
 <?xml version="1.0"?>
 <robot xmlns:xacro="http://www.ros.org/wiki/xacro">
-  <xacro:macro name="upper_rails"
-              params="parent_link xyz rpy">
+  <xacro:macro name="upper_rails" params="parent_link xyz rpy">
     <link name="upper_rails_link">
       <collision>
         <geometry>
-          <mesh filename="file://$(find ur_components_description)/meshes/upper_rails.stl" scale="0.01 0.01 0.01" />
+          <mesh filename="file://$(find ur_components_description)/meshes/upper_rails.stl" />
         </geometry>
-        <origin xyz="0.0 0.0 0.0" rpy=" ${pi/2} 0.0 ${pi/2}" />
+        <origin xyz="0.0 0.0 0.0" rpy=" 0.0 0.0 0.0" />
       </collision>
       <visual>
         <geometry>
-          <mesh filename="file://$(find ur_components_description)/meshes/upper_rails.stl" scale="0.01 0.01 0.01" />
+          <mesh filename="file://$(find ur_components_description)/meshes/upper_rails.dae" />
         </geometry>
-        <origin xyz="0.0 0.0 0.0" rpy=" ${pi/2} 0.0 ${pi/2}" />
-        <material name="Black" />
+        <origin xyz="0.0 0.0 0.0" rpy="0.0 0.0 0.0" />
       </visual>
-      <inertial>
-        <mass value="0.0000001" />
-        <inertia ixx="1.0" ixy="0.0" ixz="0.0" iyy="1.0" iyz="0.0" izz="1.0" />
-      </inertial>
     </link>
     <joint name="${parent_link}_to_upper_rails_link_joint" type="fixed">
@@ -27,7 +21,4 @@
       <child link="upper_rails_link" />
     </joint>
-    <gazebo reference="upper_rails_link">
-      <material>Gazebo/Black</material>
-    </gazebo>
   </xacro:macro>
 </robot>
