Commit message: add ur3e pkg instead of ur3

File: ur3e_moveit_config/urdf/panther_ur3e.urdf.xacro (robot description, xacro)
@@ -1,4 +1,4 @@
 <?xml version='1.0'?>
-<robot name="panther_ur3" xmlns:xacro="http://www.ros.org/wiki/xacro">
+<robot name="panther_ur3e" xmlns:xacro="http://www.ros.org/wiki/xacro">
   <xacro:arg name="use_gpu" default="false" />
   <xacro:arg name="dual_bat" default="false" />
@@ -6,5 +6,5 @@
   <!-- Robot -->
   <xacro:include filename="$(find panther_description)/urdf/panther_macro.urdf.xacro" ns="husarion" />
-  <xacro:include filename="$(find ur_description)/urdf/inc/ur3_macro.xacro" ns="universal_robot" />
+  <xacro:include filename="$(find ur_description)/urdf/inc/ur3e_macro.xacro" ns="universal_robot" />
   <xacro:include filename="$(find ur_components_description)/urdf/mounting_plate.urdf.xacro" ns="mounting_plate" />
   <xacro:include filename="$(find ur_components_description)/urdf/upper_rails.urdf.xacro" ns="rails" />
@@ -21,10 +21,10 @@
     xyz="-0.095 0.0975 0.05"
     rpy="0.0 0.0 0.0" />
-  <joint name="ur_mounting_plate_to_ur3_link_joint" type="fixed">
+  <joint name="ur_mounting_plate_to_ur3e_link_joint" type="fixed">
     <origin xyz="0.0 0.0 0.0" rpy="0.0 0.0 ${pi/2}" />
     <parent link="ur_mounting_plate_link" />
-    <child link="panther_ur3_base_link" />
+    <child link="panther_ur3e_base_link" />
   </joint>
-  <xacro:universal_robot.ur3_robot prefix="panther_ur3_" />
+  <xacro:universal_robot.ur3e_robot prefix="panther_ur3e_" />
   <!-- Components -->
   <xacro:include filename="$(find panther_description)/urdf/components/external_antenna.urdf.xacro" ns="antena" />
